File: Arduino/2020/sketch_jul21a/Glorious Krunk.brd (EAGLE design)
At the start: 68.6 x 53.3 mm, 26 parts

Commit message: modified:   Arduino/2020/sketch_jul21a/Glorious Krunk.brd 	modified:   Arduino/2020/sketch_jul21a/Glorious Krunk.ino 	modified:   Arduino/2020/sketch_jul21a/Glorious Krunk.png 	modified:   Arduino/2020/sketch_jul21a/bom.csv
Parts:
- added PIEZO2: (no value), AUTODESK_CIRCUITS_BREADBOARD:PIEZO-22MM
Connections:
- removed net N$1 (its old number): R1.1, U1.GND..
- new net N$16: PIEZO2.P$1, U1.10
- new net N$17: PIEZO2.P$2, R1.1, U1.GND..
- new net N$18: U1.GND.
